File: keybored.kicad_pcb (KiCad board)
At the start: 2 copper layers, 158 parts, among them J1 USB_C_Receptacle_USB2.0, K1 KEYSW, K10 KEYSW, K11 KEYSW, K12 KEYSW, K13 KEYSW, K14 KEYSW, K15 KEYSW, K16 KEYSW, K17 KEYSW, K18 KEYSW, K19 KEYSW, K2 KEYSW, K20 KEYSW, K21 KEYSW, K22 KEYSW, K23 KEYSW, K24 KEYSW, K25 KEYSW, K26 KEYSW, K27 KEYSW, K28 KEYSW, K29 KEYSW, K3 KEYSW, K30 KEYSW, K31 KEYSW, K32 KEYSW, K33 KEYSW, K34 KEYSW, K35 KEYSW, K36 KEYSW, K37 KEYSW, K38 KEYSW, K39 KEYSW, K4 KEYSW, K40 KEYSW, K41 KEYSW, K42 KEYSW, K43 KEYSW, K44 KEYSW, K45 KEYSW, K46 KEYSW, K47 KEYSW, K48 KEYSW, K49 KEYSW, K5 KEYSW, K50 KEYSW, K51 KEYSW, K52 KEYSW, K53 KEYSW, K54 KEYSW, K55 KEYSW, K56 KEYSW, K57 KEYSW, K58 KEYSW, K59 KEYSW, K6 KEYSW, K60 KEYSW, K61 KEYSW, K62 KEYSW, K63 KEYSW, K64 KEYSW, K65 KEYSW, K66 KEYSW, K67 KEYSW, K68 KEYSW, K69 KEYSW, K7 KEYSW, K8 KEYSW, K9 KEYSW, SW1 SW_PUSH, SW2 Rot_Enc_Sw, U1 ATMEGA32U4, U2 SSD1306, Y1 Crystal

Commit message: Key layout done
Parts:
- added REF**: Stabilizer_MX_2u, keyswitches:Stabilizer_MX_2u, F.Cu at (92.9, 123.8)
- added REF**: Stabilizer_MX_2u, keyswitches:Stabilizer_MX_2u, F.Cu at (335.8, 104.6)
- added REF**: Stabilizer_MX_2u, keyswitches:Stabilizer_MX_2u, F.Cu at (338.1, 66.7)
- moved K16 557.0 mm to (109.5, 85.7)
- moved K30 497.8 mm to (114.3, 104.8)
- moved K19 481.6 mm to (166.7, 85.7)
- moved K44 470.4 mm to (123.8, 123.8)
- moved K17 467.0 mm to (128.6, 85.7)
- moved K18 464.5 mm to (147.6, 85.7)
- moved K31 460.5 mm to (133.3, 104.8)
- moved K58 455.4 mm to (107.2, 142.9)
- moved K57 440.8 mm to (83.3, 142.9)
- moved K9 433.5 mm to (233.4, 66.7)
- moved K32 423.8 mm to (152.4, 104.8)
- moved K35 423.5 mm to (209.6, 104.8)
- moved K59 411.6 mm to (131.0, 142.9)
- moved K7 409.2 mm to (195.3, 66.7)
- moved K5 402.6 mm to (157.2, 66.7)
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
Commit message: Diode layout and row routing
Parts:
- removed the REF** at (92.9, 123.8)
- removed the REF** at (335.8, 104.6)
- removed the REF** at (338.1, 66.7)
- added REF**: Stabilizer_MX_2u, keyswitches:Stabilizer_MX_2u, F.Cu at (326.2, 114.3)
- added REF**: Stabilizer_MX_2u, keyswitches:Stabilizer_MX_2u, F.Cu at (323.9, 152.4)
- added REF**: Stabilizer_MX_2u, keyswitches:Stabilizer_MX_2u, F.Cu at (81.0, 171.4)
- C1, C2, C3, C4, C5: footprint keyboard_parts:D_SOD123_axial -> Capacitor_SMD:C_0805_2012Metric_Pad1.15x1.40mm_HandSolder
- D1, D10, D11, D12, D13, D14, D15, D16, D17, D18, D19, D2, D20, D21, D22, D23, D24, D25, D26, D27, D28, D29, D3, D30, D31, D32, D33, D34, D35, D36, D37, D38, D39, D4, D40, D41, D42, D43, D44, D45, D46, D47, D48, D49, D5, D50, D51, D52, D53, D54, D55, D56, D57, D58, D59, D6, D60, D61, D62, D63, D64, D65, D66, D67, D68, D69, D7, D70, D8, D9: footprint keyboard_parts:D_SOD123_axial -> keybored:DO-35_SOD27_5.08mm
- K1, K10, K11, K12, K13, K14, K15, K16, K17, K18, K19, K2, K20, K21, K22, K23, K24, K25, K26, K27, K28, K29, K3, K30, K31, K32, K33, K34, K35, K36, K37, K38, K39, K4, K40, K41, K42, K43, K44, K45, K46, K47, K48, K49, K5, K50, K51, K52, K53, K54, K55, K56, K57, K58, K59, K6, K60, K61, K62, K63, K64, K65, K66, K67, K68, K69, K7, K8, K9: footprint keyswitches:Kailh_socket_PG1350 -> keyswitches:Kailh_socket_MX
- moved D16 508.4 mm to (101.2, 93.8), turned to 270 degrees
- moved D45 499.4 mm to (109.5, 92.2), turned to 270 degrees
- moved D1 490.8 mm to (76.5, 92.2), turned to 270 degrees
- moved D2 490.8 mm to (104.0, 95.2), turned to 270 degrees
- moved D32 483.9 mm to (123.2, 93.8), turned to 270 degrees
- moved D30 477.6 mm to (98.5, 92.2), turned to 270 degrees
- moved D3 466.3 mm to (117.8, 96.8), turned to 270 degrees
- moved D29 465.9 mm to (82.0, 95.2), turned to 270 degrees
- moved D31 462.9 mm to (112.2, 93.8), turned to 270 degrees
- moved D33 461.6 mm to (134.2, 93.8), turned to 270 degrees
- moved D18 461.6 mm to (126.0, 95.2), turned to 270 degrees
- moved D17 460.2 mm to (115.0, 95.2), turned to 270 degrees
- moved D34 455.9 mm to (148.0, 95.2), turned to 270 degrees
- moved D70 450.9 mm to (106.8, 96.8), turned to 270 degrees
- moved D49 450.2 mm to (156.2, 93.8), turned to 270 degrees
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Routing:
- net col8: track 0.00 -> 236.3 mm
- net col1: track 0.00 -> 140.4 mm
- net col6: track 0.00 -> 140.2 mm
- net col9: track 0.00 -> 136.2 mm
- net col3: track 0.00 -> 135.3 mm
- net col4: track 0.00 -> 135.2 mm
- net col2: track 0.00 -> 133.3 mm
- net col0: track 0.00 -> 127.1 mm
- net Net-(D59-Pad2): track 0.00 -> 125.1 mm, vias 0 -> 1
- net Net-(D57-Pad2): track 0.00 -> 121.4 mm, vias 0 -> 1
- net col5: track 0.00 -> 118.2 mm
- net Net-(D58-Pad2): track 0.00 -> 106.4 mm, vias 0 -> 1
- net Net-(D45-Pad2): track 0.00 -> 101.2 mm, vias 0 -> 1
- net Net-(D44-Pad2): track 0.00 -> 100.7 mm, vias 0 -> 1
- net Net-(D46-Pad2): track 0.00 -> 94.6 mm, vias 0 -> 1
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Other:
- board outline added: 316.7 x 133.3 mm

Commit message: Finished PCB routing rev 1
Parts:
- removed D42, D55, D56: D, keybored:DO-35_SOD27_5.08mm
- removed K42, K55, K56: KEYSW, keyswitches:Kailh_socket_MX
- removed REF** (x3): Stabilizer_MX_2u, keyswitches:Stabilizer_MX_2u
- added C10: 0.1u, Capacitor_SMD:C_0805_2012Metric_Pad1.15x1.40mm_HandSolder, F.Cu at (293.2, 94.5)
- added C11: 0.1u, Capacitor_SMD:C_0805_2012Metric_Pad1.15x1.40mm_HandSolder, F.Cu at (280.0, 80.2)
- added C13: 4.7u, Capacitor_SMD:C_0805_2012Metric_Pad1.15x1.40mm_HandSolder, F.Cu at (352.2, 79.8)
- added C6: 0.1u, Capacitor_SMD:C_0805_2012Metric_Pad1.15x1.40mm_HandSolder, F.Cu at (271.9, 92.3)
- added C7: 0.1u, Capacitor_SMD:C_0805_2012Metric_Pad1.15x1.40mm_HandSolder, F.Cu at (287.0, 102.0)
- added C8: 0.1u, Capacitor_SMD:C_0805_2012Metric_Pad1.15x1.40mm_HandSolder, F.Cu at (293.2, 89.8)
- added C9: 0.1u, Capacitor_SMD:C_0805_2012Metric_Pad1.15x1.40mm_HandSolder, F.Cu at (288.0, 83.0)
- added R10: 4.7k, Resistor_SMD:R_0805_2012Metric_Pad1.15x1.40mm_HandSolder, F.Cu at (346.4, 93.6)
- added R9: 4.7k, Resistor_SMD:R_0805_2012Metric_Pad1.15x1.40mm_HandSolder, F.Cu at (346.4, 96.4)
- U2: value SSD1306 -> SSD1306-Display_Graphic; footprint Connector_PinHeader_1.00mm:PinHeader_1x04_P1.00mm_Vertical -> keybored:SSD1306_OLED_128x32_0.91_inch
- moved K63 121.5 mm to (361.9, 114.3)
- moved D63 115.4 mm to (350.0, 126.4)
- moved SW2 36.4 mm to (364.3, 85.4), turned to 270 degrees
- moved C2 31.9 mm to (269.4, 83.1), turned to 90 degrees
- moved R5 29.2 mm to (272.0, 100.5), turned to 0 degrees
- moved C1 24.2 mm to (277.9, 82.4), turned to 270 degrees
- moved Y1 23.4 mm to (273.5, 82.7), turned to 180 degrees
- moved U2 22.6 mm to (341.8, 88.5)
- moved C3 17.8 mm to (290.2, 83.0), turned to 90 degrees
- moved D68 11.7 mm to (347.7, 128.6)
- moved D69 10.8 mm to (345.3, 131.0)
- moved C5 9.45 mm to (344.6, 117.2), turned to 180 degrees
- moved SW1 7.79 mm to (306.6, 79.1)
- moved R6 7.40 mm to (293.8, 80.9), turned to 90 degrees
- moved R7 7.16 mm to (344.6, 111.2), turned to 180 degrees
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Connections:
- U2 pad 1: (no net) -> GND
- U2 pad 2: (no net) -> VCC
- U2 pad 3: (no net) -> I2C_SCL
- U2 pad 4: (no net) -> I2C_SDA
Routing:
- net row6: track 0.00 -> 459.0 mm, vias 0 -> 4
- net row5: track 0.00 -> 375.6 mm, vias 0 -> 5
- net row4: track 0.00 -> 370.6 mm, vias 0 -> 5
- net row2: track 0.00 -> 276.4 mm, vias 0 -> 4
- net rotSw2: track 0.00 -> 274.5 mm, vias 0 -> 1
- net row3: track 0.00 -> 272.6 mm, vias 0 -> 4
- net row1: track 0.00 -> 269.5 mm, vias 0 -> 3
- net row0: track 0.00 -> 261.5 mm, vias 0 -> 3
- net col6: track 140.2 -> 381.9 mm, vias 0 -> 1
- net col4: track 135.2 -> 362.8 mm, vias 0 -> 1
- net col8: track 236.3 -> 444.8 mm, vias 0 -> 1
- net col2: track 133.3 -> 340.8 mm, vias 0 -> 1
- net Net-(D64-Pad2): track 2.37 -> 199.8 mm
- net Net-(D66-Pad2): track 2.33 -> 193.1 mm
- net Net-(D65-Pad2): track 2.31 -> 186.6 mm
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- added copper zone on B.Cu, net GND
- added copper zone on F.Cu, net GND

Commit message: Updated PCB image
Routing:
- net GND: track 40.3 -> 34.2 mm, vias 13 -> 14

Commit message: Major pcb changes
- now uses a dual footprint for switches
- added ARGB support
- added stabilizer holes
- added header pin support for ISP
Parts:
- removed K67, K68, K69: KEYSW, keyswitches:Kailh_socket_MX
- added D68: WS2812B, LED_SMD:LED_WS2812B_PLCC4_5.0x5.0mm_P3.2mm, B.Cu at (292.9, 104.8)
- added D69: WS2812B, LED_SMD:LED_WS2812B_PLCC4_5.0x5.0mm_P3.2mm, B.Cu at (254.8, 181.0)
- added D70: WS2812B, LED_SMD:LED_WS2812B_PLCC4_5.0x5.0mm_P3.2mm, B.Cu at (85.9, 142.6)
- added D71: WS2812B, LED_SMD:LED_WS2812B_PLCC4_5.0x5.0mm_P3.2mm, B.Cu at (254.8, 104.8)
- added D72: WS2812B, LED_SMD:LED_WS2812B_PLCC4_5.0x5.0mm_P3.2mm, B.Cu at (331.0, 104.8)
- added D73: WS2812B, LED_SMD:LED_WS2812B_PLCC4_5.0x5.0mm_P3.2mm, B.Cu at (215.5, 181.0)
- added D74: WS2812B, LED_SMD:LED_WS2812B_PLCC4_5.0x5.0mm_P3.2mm, B.Cu at (100.0, 104.8)
- added D75: WS2812B, LED_SMD:LED_WS2812B_PLCC4_5.0x5.0mm_P3.2mm, B.Cu at (346.3, 142.6)
- added D76: WS2812B, LED_SMD:LED_WS2812B_PLCC4_5.0x5.0mm_P3.2mm, B.Cu at (176.2, 181.0)
- added D77: WS2812B, LED_SMD:LED_WS2812B_PLCC4_5.0x5.0mm_P3.2mm, B.Cu at (138.1, 104.8)
- added D78: WS2812B, LED_SMD:LED_WS2812B_PLCC4_5.0x5.0mm_P3.2mm, B.Cu at (331.0, 181.0)
- added D79: WS2812B, LED_SMD:LED_WS2812B_PLCC4_5.0x5.0mm_P3.2mm, B.Cu at (138.1, 181.0)
- added D80: WS2812B, LED_SMD:LED_WS2812B_PLCC4_5.0x5.0mm_P3.2mm, B.Cu at (176.2, 104.8)
- added D81: WS2812B, LED_SMD:LED_WS2812B_PLCC4_5.0x5.0mm_P3.2mm, B.Cu at (292.9, 181.0)
- added D82: WS2812B, LED_SMD:LED_WS2812B_PLCC4_5.0x5.0mm_P3.2mm, B.Cu at (100.0, 181.0)
- added D83: WS2812B, LED_SMD:LED_WS2812B_PLCC4_5.0x5.0mm_P3.2mm, B.Cu at (215.5, 105.0)
- added J2: AVR-ISP-6, Connector_PinHeader_2.54mm:PinHeader_2x03_P2.54mm_Vertical, F.Cu at (291.9, 84.0)
- added J3: Conn_01x03, Connector_PinHeader_2.54mm:PinHeader_1x03_P2.54mm_Vertical, B.Cu at (311.1, 95.9)
- added J4: Conn_01x03, Connector_PinHeader_2.54mm:PinHeader_1x03_P2.54mm_Vertical, B.Cu at (255.2, 97.8)
- added K42: KEYSW, keyswitches:Kailh_socket_MX_optional, F.Cu at (81.0, 171.4)
- added K55: KEYSW, keyswitches:Kailh_socket_MX_optional, F.Cu at (95.2, 190.5)
- added K56: KEYSW, keyswitches:Kailh_socket_MX_optional, F.Cu at (119.1, 190.5)
- added R7: 330, Resistor_SMD:R_0805_2012Metric_Pad1.15x1.40mm_HandSolder, F.Cu at (295.3, 100.2)
- added REF**: MountingHole_2.2mm_M2_Pad, MountingHole:MountingHole_2.2mm_M2_Pad, F.Cu at (61.9, 78.6)
- added REF**: MountingHole_2.2mm_M2_Pad, MountingHole:MountingHole_2.2mm_M2_Pad, F.Cu at (61.9, 102.4)
- added REF**: MountingHole_2.2mm_M2_Pad, MountingHole:MountingHole_2.2mm_M2_Pad, F.Cu at (369.1, 102.4)
- added REF**: MountingHole_2.2mm_M2_Pad, MountingHole:MountingHole_2.2mm_M2_Pad, F.Cu at (369.1, 78.6)
- added REF**: Stabilizer_MX_2u, keyswitches:Stabilizer_MX_2u, F.Cu at (81.0, 171.4)
- added REF**: Stabilizer_MX_2u, keyswitches:Stabilizer_MX_2u, F.Cu at (323.9, 152.4)
- added REF**: Stabilizer_MX_2u, keyswitches:Stabilizer_MX_2u, F.Cu at (326.2, 114.3)
- added REF**: MountingHole_2.2mm_M2_Pad, MountingHole:MountingHole_2.2mm_M2_Pad, F.Cu at (308.0, 122.0)
- added REF**: MountingHole_2.2mm_M2_Pad, MountingHole:MountingHole_2.2mm_M2_Pad, F.Cu at (308.0, 154.8)
- added REF**: MountingHole_2.2mm_M2_Pad, MountingHole:MountingHole_2.2mm_M2_Pad, F.Cu at (361.9, 173.8)
- added REF**: MountingHole_2.2mm_M2_Pad, MountingHole:MountingHole_2.2mm_M2_Pad, F.Cu at (309.6, 193.0)
- added REF**: MountingHole_2.2mm_M2_Pad, MountingHole:MountingHole_2.2mm_M2_Pad, F.Cu at (210.0, 193.0)
- added REF**: MountingHole_2.2mm_M2_Pad, MountingHole:MountingHole_2.2mm_M2_Pad, F.Cu at (135.7, 193.0)
- added REF**: MountingHole_2.2mm_M2_Pad, MountingHole:MountingHole_2.2mm_M2_Pad, F.Cu at (98.0, 173.8)
- added REF**: MountingHole_2.2mm_M2_Pad, MountingHole:MountingHole_2.2mm_M2_Pad, F.Cu at (86.0, 133.3)
- K1, K10, K11, K12, K13, K14, K15, K16, K17, K18, K19, K2, K20, K21, K22, K23, K24, K25, K26, K27, K28, K29, K3, K30, K31, K32, K33, K34, K35, K36, K37, K38, K39, K4, K40, K41, K43, K44, K45, K46, K47, K48, K49, K5, K50, K51, K52, K53, K54, K57, K58, K59, K6, K60, K61, K62, K63, K64, K65, K66, K7, K8, K9: footprint keyswitches:Kailh_socket_MX -> keyswitches:Kailh_socket_MX_optional
- moved K54 238.9 mm to (71.4, 190.5)
- moved K60 187.5 mm to (361.9, 114.3)
- moved K59 173.8 mm to (292.9, 190.5)
- moved K58 169.1 mm to (264.3, 190.5)
- moved K57 119.1 mm to (190.5, 190.5)
- moved K63 81.0 mm to (361.9, 195.3)
- moved K65 64.8 mm to (361.9, 133.3)
- moved K61 59.7 mm to (323.9, 195.3)
- moved K62 50.2 mm to (342.9, 195.3)
- moved K66 42.9 mm to (361.9, 152.4)
- moved K43 31.0 mm to (111.9, 171.4)
- moved K64 26.9 mm to (342.9, 176.2)
- moved K53 26.2 mm to (309.6, 171.4)
- moved K45 19.1 mm to (150.0, 171.4)
- moved K47 19.1 mm to (188.1, 171.4)
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- renumbered C6 to C1, C13 to C10, C4 to C11, C5 to C12, C7 to C2, C8 to C3, C9 to C4, C10 to C5, C1 to C6, C11 to C7, C2 to C8, C3 to C9, D43 to D42, D44 to D43, D45 to D44, D46 to D45, D47 to D46, D48 to D47, D49 to D48, D50 to D49, D51 to D50, D52 to D51, D53 to D52, D54 to D53, D57 to D54, D58 to D55, D59 to D56, D60 to D57, D61 to D58, D62 to D59, D63 to D60, D64 to D61, D65 to D62, D66 to D63, D67 to D64, D68 to D65, D69 to D66, D70 to D67, R9 to R10, R10 to R11, R7 to R8, R8 to R9
Connections:
- D42 pad 2: Net-(D43-Pad2) -> Net-(D42-Pad2)
- D43 pad 2: Net-(D44-Pad2) -> Net-(D43-Pad2)
- D44 pad 2: Net-(D45-Pad2) -> Net-(D44-Pad2)
- D45 pad 2: Net-(D46-Pad2) -> Net-(D45-Pad2)
- D46 pad 2: Net-(D47-Pad2) -> Net-(D46-Pad2)
- D47 pad 2: Net-(D48-Pad2) -> Net-(D47-Pad2)
- D48 pad 2: Net-(D49-Pad2) -> Net-(D48-Pad2)
- D49 pad 2: Net-(D50-Pad2) -> Net-(D49-Pad2)
- D50 pad 2: Net-(D51-Pad2) -> Net-(D50-Pad2)
- D51 pad 2: Net-(D52-Pad2) -> Net-(D51-Pad2)
- D52 pad 2: Net-(D53-Pad2) -> Net-(D52-Pad2)
- D53 pad 2: Net-(D54-Pad2) -> Net-(D53-Pad2)
- D54 pad 2: Net-(D57-Pad2) -> Net-(D54-Pad2)
- D55 pad 2: Net-(D58-Pad2) -> Net-(D55-Pad2)
- D56 pad 2: Net-(D59-Pad2) -> Net-(D56-Pad2)
- D57 pad 2: Net-(D60-Pad2) -> Net-(D57-Pad2)
- D58 pad 2: Net-(D61-Pad2) -> Net-(D58-Pad2)
- D59 pad 2: Net-(D62-Pad2) -> Net-(D59-Pad2)
- D60 pad 2: Net-(D63-Pad2) -> Net-(D60-Pad2)
- D61 pad 2: Net-(D64-Pad2) -> Net-(D61-Pad2)
- D62 pad 2: Net-(D65-Pad2) -> Net-(D62-Pad2)
- D63 pad 2: Net-(D66-Pad2) -> Net-(D63-Pad2)
- D64 pad 2: Net-(D67-Pad2) -> Net-(D64-Pad2)
- D65 pad 2: Net-(D68-Pad2) -> Net-(D65-Pad2)
- D66 pad 2: Net-(D69-Pad2) -> Net-(D66-Pad2)
- K49 pad 1: col6 -> col7
- K54 pad 1: col7 -> col8
- K61 pad 1: col8 -> col9
- K62 pad 1: col8 -> col9
- K63 pad 1: col8 -> col9
- U1 pad 1: Net-(U1-Pad1) -> RGB_IN
Routing:
- net VCC: track 152.9 -> 956.4 mm, vias 0 -> 5
- net Net-(D63-Pad2): track 23.9 -> 210.4 mm, vias 1 -> 0
- net Net-(D67-Pad2): track 162.3 -> 0.00 mm, vias 1 -> 0
- net Net-(D65-Pad2): track 186.6 -> 25.1 mm, vias 1 -> 0
- net Net-(D66-Pad2): track 193.1 -> 39.3 mm, vias 1 -> 0
- net col4: track 362.8 -> 508.1 mm
- net Net-(D56-Pad2): track 0.00 -> 142.3 mm
- net col6: track 381.9 -> 523.1 mm
- net col2: track 340.8 -> 480.8 mm
- net col8: track 444.8 -> 583.0 mm
- net col3: track 216.8 -> 340.6 mm
- net Net-(D55-Pad2): track 0.00 -> 121.1 mm
- net col9: track 245.2 -> 363.8 mm
- net col0: track 244.1 -> 355.4 mm
- net col7: track 236.2 -> 343.8 mm
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Other:
- board text added: "+5V"
- board text added: "Din"
- board text added: "Dout"
- board text added: "GND"

Commit message: Add plate, updates to PCB
Parts:
- removed the REF** at (61.9, 102.4)
- removed the REF** at (369.1, 102.4)
- removed the REF** at (369.1, 78.6)
- added REF**: MountingHole_2.2mm_M2_Pad, MountingHole:MountingHole_2.2mm_M2_Pad, F.Cu at (61.9, 97.6)
- added REF**: MountingHole_2.2mm_M2_Pad, MountingHole:MountingHole_2.2mm_M2_Pad, F.Cu at (340.5, 97.6)
- added REF**: MountingHole_2.2mm_M2_Pad, MountingHole:MountingHole_2.2mm_M2_Pad, F.Cu at (314.3, 78.6)
- J2: value AVR-ISP-6 -> ISP
- moved SW2 17.9 mm to (369.5, 90.0)
- moved R4 11.8 mm to (321.0, 79.5), turned to 0 degrees
- moved R3 9.42 mm to (321.0, 77.0), turned to 0 degrees
- moved J1 8.68 mm to (336.9, 74.0)
- moved C10 7.45 mm to (344.8, 80.0)
- moved R2 6.58 mm to (329.0, 77.0), turned to 0 degrees
- moved U2 4.40 mm to (326.6, 84.0)
- moved R11 4.37 mm to (331.1, 89.1)
- moved R10 4.37 mm to (331.1, 91.9)
- moved J2 4.35 mm to (291.9, 79.7)
- moved SW1 3.80 mm to (306.3, 78.4)
- moved R1 2.79 mm to (329.0, 79.5), turned to 0 degrees
- moved K12 0.74 mm to (278.6, 114.3)
- moved K60 0.10 mm to (361.9, 114.3)
Routing:
- net VCC: track 956.4 -> 1035.8 mm, vias 5 -> 8
- net row6: track 428.0 -> 457.3 mm
- net Net-(J1-PadB5): track 32.3 -> 6.83 mm
- net GND: track 45.9 -> 63.5 mm, vias 34 -> 38
- net rotSw2: track 255.6 -> 273.0 mm
- net Net-(R4-Pad1): track 65.1 -> 48.3 mm
- net Net-(R9-Pad2): track 35.7 -> 50.3 mm
- net Net-(R8-Pad1): track 22.6 -> 36.2 mm
- net Net-(J1-PadA5): track 22.8 -> 10.5 mm, vias 0 -> 1
- net Net-(R3-Pad1): track 63.6 -> 51.6 mm
- net col8: track 583.0 -> 574.5 mm
- net col9: track 363.8 -> 371.7 mm
- net USB_D-: track 24.1 -> 20.8 mm
- net I2C_SDA: track 81.5 -> 84.3 mm
- net Net-(D70-Pad4): track 83.9 -> 81.4 mm
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Other:
- net class PWR added: clearance 0.2, trace_width 0.35, via_dia 1, via_drill 0.4

Commit message: Updates to PCB + Plate
- plate dimensions fixed
- cutouts for stabilizers added
- spacebar stabilizer holes added to PCB
- moved RGB LEDs on PCB
Parts:
- removed the REF** at (308.0, 154.8)
- removed the REF** at (98.0, 173.8)
- added G***: LOGO, keybored:sadge_decal, B.Cu at (162.4, 195.2)
- added REF**: floppy_disks_2, keybored:floppy_disks_2, F.Cu at (74.5, 84.0)
- added REF**: MountingHole_2.2mm_M2_Pad, MountingHole:MountingHole_2.2mm_M2_Pad, F.Cu at (100.0, 171.4)
- added REF**: Fuse_0805, Fuse:Fuse_0805_2012Metric_Pad1.15x1.40mm_HandSolder, B.Cu at (340.0, 82.2)
- added REF**: JST-SR-4, random-keyboard-parts:JST-SR-4, B.Cu at (347.0, 90.0)
- added REF**: MX_Stabilizers_6.25u, keybored:MX_Stabilizers_6.25u, F.Cu at (190.5, 190.5)
- added REF**: MountingHole_2.2mm_M2_Pad, MountingHole:MountingHole_2.2mm_M2_Pad, F.Cu at (304.8, 154.8)
- moved D77 4.76 mm to (133.3, 104.8)
- moved D79 4.76 mm to (133.3, 181.0)
- moved D81 4.76 mm to (297.7, 181.0)
- moved REF** 4.76 mm to (131.0, 193.0)
- moved C10 1.55 mm to (346.0, 79.2)
Routing:
- net USB_D+: track 21.5 -> 37.2 mm, vias 0 -> 1
- net USB_D-: track 20.8 -> 36.0 mm, vias 0 -> 1
- net VCC: track 1035.8 -> 1050.1 mm, vias 8 -> 9
- net col2: track 480.8 -> 473.0 mm
- net col3: track 340.6 -> 332.8 mm
- net col4: track 508.1 -> 500.3 mm
- net col5: track 314.9 -> 307.1 mm
- net col6: track 523.1 -> 515.3 mm
- net col7: track 343.8 -> 336.0 mm
- net col8: track 574.5 -> 566.7 mm
- net col9: track 371.7 -> 363.9 mm
- net Net-(D76-Pad2): track 36.5 -> 42.3 mm
- net Net-(D79-Pad2): track 37.2 -> 32.0 mm
- net Net-(D74-Pad2): track 54.3 -> 49.5 mm
- net Net-(D78-Pad2): track 41.2 -> 36.5 mm
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Other:
- board text added: "Prototype Rev. 1"
- board text added: "Staccato 65"
- board text added: "USB"

Commit message: Final touches on PCB and Plate
- added decals and memes on PCB + plate
- copper fill added for plate
- final commit before prototype order
Parts:
- added REF**: square_diagonal, keybored:square_diagonal, F.Cu at (75.0, 80.6)
- REF**: moved to B.Cu
- moved REF** 180.5 mm to (255.0, 83.8), turned to 180 degrees
- moved G*** 2.55 mm to (160.5, 193.5)
Routing:
- net row6: track 460.3 -> 413.8 mm, vias 4 -> 5
- net row5: track 378.4 -> 367.4 mm
- net row3: track 267.6 -> 257.7 mm
- net row4: track 372.8 -> 363.1 mm
- net row2: track 270.8 -> 261.8 mm
- net row1: track 263.3 -> 256.9 mm
- net row0: track 254.7 -> 249.0 mm
Other:
- board text added: "!"
- board text added: "BEWARE ESD"
- board text added: "Eric Li"
- board text added: "Everything not saved will be lost."
- board text added: "HIGH VOLTAGE"
- board text added: "NOT MACHINE WASHABLE"
- board text added: "Nah, I'm just messing with ya."
- board text added: "PCB Designed by"
