File: keybored_plate/keybored_plate.kicad_pcb (KiCad board)
At the start: 2 copper layers, 328.7 x 111.1 mm, 15 parts

Commit message: Updates to PCB + Plate
- plate dimensions fixed
- cutouts for stabilizers added
- spacebar stabilizer holes added to PCB
- moved RGB LEDs on PCB
Parts:
- removed the REF** at (210.4, 210.7)
- removed the REF** at (357.2, 176.2)
- removed the REF** at (304.8, 195.4)
- removed the REF** at (50.3, 169.6)
- removed the REF** at (371.2, 169.6)
- removed the REF** at (371.2, 111.0)
- removed the REF** at (50.3, 111.0)
- removed the REF** at (313.5, 217.2)
- removed the REF** at (109.1, 210.9)
- removed the REF** at (81.2, 135.7)
- removed the REF** at (93.2, 176.2)
- removed the REF** at (131.0, 195.4)
- removed the REF** at (303.2, 157.2)
- removed the REF** at (205.2, 195.4)
- removed the REF** at (303.2, 124.4)
- added REF**: MountingHole_2.2mm_M2_Pad, MountingHole:MountingHole_2.2mm_M2_Pad, F.Cu at (316.7, 208.6)
- added REF**: MountingHole_2.2mm_M2_Pad, MountingHole:MountingHole_2.2mm_M2_Pad, F.Cu at (361.9, 173.8)
- added REF**: MountingHole_2.2mm_M2_Pad, MountingHole:MountingHole_2.2mm_M2_Pad, F.Cu at (308.0, 122.0)
- added REF**: MountingHole_2.2mm_M2_Pad, MountingHole:MountingHole_2.2mm_M2_Pad, F.Cu at (210.0, 193.0)
- added REF**: MountingHole_2.2mm_M2_Pad, MountingHole:MountingHole_2.2mm_M2_Pad, F.Cu at (375.5, 113.6)
- added REF**: MountingHole_2.2mm_M2_Pad, MountingHole:MountingHole_2.2mm_M2_Pad, B.Cu at (55.3, 167.3)
- added REF**: MountingHole_2.2mm_M2_Pad, MountingHole:MountingHole_2.2mm_M2_Pad, F.Cu at (114.2, 208.6)
- added REF**: MountingHole_2.2mm_M2_Pad, MountingHole:MountingHole_2.2mm_M2_Pad, F.Cu at (215.5, 208.6)
- added REF**: MountingHole_2.2mm_M2_Pad, MountingHole:MountingHole_2.2mm_M2_Pad, F.Cu at (100.0, 171.4)
- added REF**: MountingHole_2.2mm_M2_Pad, MountingHole:MountingHole_2.2mm_M2_Pad, F.Cu at (86.0, 133.3)
- added REF**: MountingHole_2.2mm_M2_Pad, MountingHole:MountingHole_2.2mm_M2_Pad, F.Cu at (131.0, 192.9)
- added REF**: MountingHole_2.2mm_M2_Pad, MountingHole:MountingHole_2.2mm_M2_Pad, F.Cu at (309.6, 193.0)
- added REF**: MountingHole_2.2mm_M2_Pad, MountingHole:MountingHole_2.2mm_M2_Pad, F.Cu at (375.6, 167.3)
- added REF**: MountingHole_2.2mm_M2_Pad, MountingHole:MountingHole_2.2mm_M2_Pad, F.Cu at (304.8, 154.8)
- added REF**: MountingHole_2.2mm_M2_Pad, MountingHole:MountingHole_2.2mm_M2_Pad, F.Cu at (55.3, 113.6)
Other:
- board size 328.7 x 111.1 mm -> 328.1 x 108 mm
- board text added: "Middle Tab: X: 0.3 (too left)"
- board text added: "Tab: X: 0.14 (too right)"
- board text added: "Tab: Y: 0.08 (too high)"
- board text added: "X: 0.125 (too right), Y: 0.05 (too high)"

Commit message: Final touches on PCB and Plate
- added decals and memes on PCB + plate
- copper fill added for plate
- final commit before prototype order
Routing:
- added copper zone on B.Cu, net (none)
- added copper zone on F.Cu, net (none)
Other:
- board text added: "Case: Sagar Dighe"
- board text added: "PCB: Eric Li"
- board text added: "Prototype Rev. 1"
- board text added: "Staccato 65"
Changed lines of the file:
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@@
   (general
     (thickness 1.6)
-    (drawings 708)
+    (drawings 740)
     (tracks 0)
     (zones 0)
@@
       (outputformat 1)
       (mirror false)
-      (drillshape 1)
+      (drillshape 0)
       (scaleselection 1)
-      (outputdirectory ""))
+      (outputdirectory "gerbers/"))
   )
   (net 0 "")
@@
     )
     (pad 1 thru_hole circle (at 0 0) (size 4.4 4.4) (drill 2.2) (layers *.Cu *.Mask))
+  )
+  (gr_text "Case: Sagar Dighe " (at 186 203) (layer B.SilkS)
+    (effects (font (size 1.5 1.5) (thickness 0.3)) (justify mirror))
+  )
+  (gr_text "PCB: Eric Li " (at 189.5 200) (layer B.SilkS)
+    (effects (font (size 1.5 1.5) (thickness 0.3)) (justify mirror))
+  )
+  (gr_poly (pts (xy 225.5 187) (xy 226 187) (xy 226 185) (xy 227 185) (xy 227 188) (xy 223 188) (xy 223 185) (xy 225.5 185)) (layer F.Mask) (width 0.1))
+  (gr_line (start 228 190) (end 228 194) (layer F.Mask) (width 0.15))
+  (gr_line (start 221.5 190) (end 228 190) (layer F.Mask) (width 0.15))
+  (gr_line (start 221.5 194) (end 221.5 190) (layer F.Mask) (width 0.15))
+  (gr_line (start 220 194) (end 220 185) (layer F.Mask) (width 0.15))
+  (gr_line (start 229 194) (end 220 194) (layer F.Mask) (width 0.15))
+  (gr_line (start 225.5 240) (end 226 240) (layer Dwgs.User) (width 0.15))
+  (gr_line (start 228 239) (end 229.5 241) (layer Dwgs.User) (width 0.15))
+  (gr_line (start 226 240) (end 228 239) (layer Dwgs.User) (width 0.15))
+  (gr_line (start 226 240) (end 227 241) (layer Dwgs.User) (width 0.15))
+  (gr_line (start 228 185) (end 229 186) (layer F.Mask) (width 0.2))
+  (gr_line (start 226 240) (end 227 241) (layer Dwgs.User) (width 0.15))
+  (gr_line (start 220 185) (end 228 185) (layer F.Mask) (width 0.2))
+  (gr_line (start 229 186) (end 229 194) (layer F.Mask) (width 0.2))
+  (gr_text "Prototype Rev. 1" (at 163.31 191.5) (layer F.Cu)
+    (effects (font (size 2 2) (thickness 0.2)))
+  )
+  (gr_text "Staccato 65" (at 163.31 188) (layer F.Cu)
+    (effects (font (size 2 2) (thickness 0.2)))
+  )
+  (gr_line (start 151 185) (end 176.5 185) (layer F.Cu) (width 0.2))
+  (gr_line (start 150 195) (end 150 186) (layer F.Cu) (width 0.2))
+  (gr_line (start 151 185) (end 150 186) (layer F.Cu) (width 0.2))
+  (gr_line (start 176.5 194) (end 175.5 195) (layer F.Cu) (width 0.2))
+  (gr_line (start 176.5 185) (end 176.5 194) (layer F.Cu) (width 0.2))
+  (gr_line (start 175.5 195) (end 150 195) (layer F.Cu) (width 0.2))
+  (gr_line (start 176.5 194) (end 175.5 195) (layer F.Mask) (width 0.2))
+  (gr_line (start 150 195) (end 150 186) (layer F.Mask) (width 0.2))
+  (gr_line (start 175.5 195) (end 150 195) (layer F.Mask) (width 0.2))
+  (gr_line (start 176.5 185) (end 176.5 194) (layer F.Mask) (width 0.2))
+  (gr_line (start 151 185) (end 176.5 185) (layer F.Mask) (width 0.2))
+  (gr_line (start 151 185) (end 150 186) (layer F.Mask) (width 0.2))
+  (gr_text "Prototype Rev. 1" (at 163.31 191.5) (layer F.Mask)
+    (effects (font (size 2 2) (thickness 0.2)))
+  )
+  (gr_text "Staccato 65" (at 163.31 188) (layer F.Mask)
+    (effects (font (size 2 2) (thickness 0.2)))
   )
   (gr_line (start 305.6825 211.16875) (end 327.6825 211.16875) (layer Edge.Cuts) (width 0.05))
@@
   (gr_line (start 379.5625 174.80875) (end 379.5625 159.80875) (layer Edge.Cuts) (width 0.05))
   (gr_arc (start 378.5625 174.80875) (end 378.5625 175.80875) (angle -90) (layer Edge.Cuts) (width 0.05))
-  (gr_arc (start 378.5625 159.80875) (end 379.5625 159.80875) (angle -90.42917384) (layer Edge.Cuts) (width 0.05))
+  (gr_arc (start 378.5625 159.80875) (end 379.5625 159.80875) (angle -90) (layer Edge.Cuts) (width 0.05))
   (gr_arc (start 378.5625 104.11875) (end 379.5625 104.11875) (angle -90) (layer Edge.Cuts) (width 0.05))
   (gr_arc (start 378.5625 121.11875) (end 378.5625 122.11875) (angle -90) (layer Edge.Cuts) (width 0.05))
@@
   (gr_arc (start 336.902499 189.262501) (end 336.902499 188.262501) (angle -90) (layer Edge.Cuts) (width 0.2))
   (gr_line (start 227.4625 210.16875) (end 227.4625 207.16875) (layer Edge.Cuts) (width 0.05))
-  (gr_line (start 52.4625 175.80875) (end 57.4625 175.80875) (layer Edge.Cuts) (width 0.05))
+  (gr_line (start 52.46999 175.808722) (end 57.4625 175.80875) (layer Edge.Cuts) (width 0.05))
   (gr_line (start 203.4625 207.16875) (end 126.2025 207.16875) (layer Edge.Cuts) (width 0.05))
   (gr_line (start 102.2025 207.16875) (end 102.2025 210.16875) (layer Edge.Cuts) (width 0.05))
@@
     (effects (font (size 1.5 1.5) (thickness 0.3)))
   )
+  (zone (net 0) (net_name "") (layer F.Cu) (hatch edge 0.508)
+    (connect_pads (clearance 0.508))
+    (min_thickness 0.254)
+    (fill yes (arc_segments 32) (thermal_gap 0.508) (thermal_bridge_width 0.508))
+    (polygon
+      (pts
+        (xy 381 212) (xy 50 212) (xy 50 102) (xy 381 102)
+      )
+    )
+  )
+  (zone (net 0) (net_name "") (layer B.Cu) (hatch edge 0.508)
+    (connect_pads (clearance 0.508))
+    (min_thickness 0.254)
+    (fill yes (arc_segments 32) (thermal_gap 0.508) (thermal_bridge_width 0.508))
+    (polygon
+      (pts
+        (xy 381 212) (xy 50 212) (xy 50 102) (xy 381 102)
+      )
+    )
+  )
+  (zone (net 0) (net_name "") (layer F.Cu) (hatch edge 0.508)
+    (connect_pads (clearance 0.508))
+    (min_thickness 0.254)
+    (keepout (tracks allowed) (vias allowed) (copperpour not_allowed))
+    (fill (arc_segments 32) (thermal_gap 0.508) (thermal_bridge_width 0.508))
+    (polygon
+      (pts
+        (xy 176.5 194) (xy 175.5 195) (xy 150 195) (xy 150 186) (xy 151 185)
+        (xy 176.5 185)
+      )
+    )
+  )
+  (zone (net 0) (net_name "") (layer F.Cu) (hatch edge 0.508)
+    (connect_pads (clearance 0.508))
+    (min_thickness 0.254)
+    (keepout (tracks not_allowed) (vias not_allowed) (copperpour not_allowed))
+    (fill (arc_segments 32) (thermal_gap 0.508) (thermal_bridge_width 0.508))
+    (polygon
+      (pts
+        (xy 228 194) (xy 221.5 194) (xy 221.5 190) (xy 228 190)
+      )
+    )
+  )
+  (zone (net 0) (net_name "") (layer F.Cu) (hatch edge 0.508)
+    (connect_pads (clearance 0.508))
+    (min_thickness 0.254)
+    (keepout (tracks not_allowed) (vias not_allowed) (copperpour not_allowed))
+    (fill (arc_segments 32) (thermal_gap 0.508) (thermal_bridge_width 0.508))
+    (polygon
+      (pts
+        (xy 226 187) (xy 225.5 187) (xy 225.5 185) (xy 226 185)
+      )
+    )
+  )
 )
